File: pcb/micro10.kicad_pcb (KiCad board)
At the start: 2 copper layers, 190.5 x 87.3 mm, 57 parts, among them J1 Conn_01x08_Female, SW1 SW_Push, U1 Elite-C

Commit message: Case files
Parts:
- MX410: footprint MX_Only:MXOnly-1U-Hotswap -> MX_Only:MXOnly-1.25U-Hotswap
- moved U1 2.54 mm to (148.4, 46.7)
- moved MX410 2.38 mm to (241.3, 106.4)
Routing:
- net Col7: track 103.4 -> 106.1 mm
- net Col0: track 144.4 -> 147.0 mm
- net SDA: track 83.9 -> 86.4 mm
- net Col1: track 105.1 -> 107.7 mm
- net +5V: track 87.2 -> 89.8 mm
- net Row3: track 162.7 -> 165.3 mm
- net Col3: track 117.7 -> 115.2 mm
- net Col2: track 111.8 -> 109.2 mm
- net Row2: track 187.7 -> 190.3 mm
- net Net-(D410-Pad2): track 61.5 -> 59.2 mm
- net ENB: track 82.2 -> 84.3 mm
- net ENA: track 91.2 -> 93.1 mm
- net SCL: track 84.4 -> 85.7 mm
- net Col4: track 64.5 -> 65.7 mm
- net Col5: track 75.3 -> 76.3 mm
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