File: pcb/micro10.kicad_sch (KiCad schematic)
At the start: 54 parts, among them J1 Conn_01x08_Female, SW1 SW_Push, U1 Elite-C

Commit message: Case files
Other:
- note added: "0"
- note added: "1"
- note added: "18"
- note added: "19"
- note added: "20"
- note added: "21"
Changed lines of the file:
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@@
     (stroke (width 0) (type default) (color 0 0 0 0))
+  )
+  (text "1" (at 62.23 49.53 0)
+    (effects (font (size 1.27 1.27)) (justify left bottom))
+  )
+  (text "21" (at 66.04 59.69 0)
+    (effects (font (size 1.27 1.27)) (justify left bottom))
+  )
+  (text "0" (at 62.23 52.07 0)
+    (effects (font (size 1.27 1.27)) (justify left bottom))
+  )
+  (text "19" (at 66.04 64.77 0)
+    (effects (font (size 1.27 1.27)) (justify left bottom))
+  )
+  (text "20" (at 66.04 62.23 0)
+    (effects (font (size 1.27 1.27)) (justify left bottom))
+  )
+  (text "18" (at 66.04 67.31 0)
+    (effects (font (size 1.27 1.27)) (justify left bottom))
   )
   (global_label "Col8" (shape input) (at 82.55 68.58 0) (fields_autoplaced)
